File: eagle/CR78-GU.brd (EAGLE design)
At the start: 100.8 x 80.8 mm, 39 parts, among them Q509 2N3904, Q522 2N3904, Q523 2N3904, Q524 2N3904, Q7 2N3904

Commit message: connector for gu
Parts:
- removed C534, C535: 27n, rcl:C050-025X075
- removed C536: 56n, rcl:C050-025X075
- removed C537: 10n, rcl:C050-025X075
- removed C538: 33n, rcl:C050-025X075
- removed D521, D522, D523, D528, D529: (no value), SparkFun-DiscreteSemi:DIODE-1N4148
- removed L5: 1R (40mH), rcl:0207/5V
- removed Q509, Q524: 2N3904, 808_lt:TO92
- removed R555, R556, R557: 270k, rcl:0207/7
- removed R558, R681: 820k, rcl:0207/7
- removed R559: 10k, rcl:0207/7
- removed R560: 2M2, rcl:0207/7
- removed R561: 47k, rcl:0207/7
- removed R562: 470k, rcl:0207/7
- removed TB: 22-23-2071, con-molex:22-23-2071
- added GU: (no value), con-molex:22-23-2061
- added VR59: 100K, TR808clone:B64Y
- renumbered VR62 to VR63
Connections:
- removed net N$1: C535.2, D522.C, D528.C, R555.1
- removed net N$10: Q509.2, R561.1, R562.2
- removed net N$14: Q524.2, R557.2, R558.2, R681.1
- removed net N$2: D522.A, R558.1
- removed net N$22: C534.2, D521.C, D529.C, R556.1
- removed net N$23: D521.A, R557.1
- removed net N$25: D528.A, D529.A, TB.3
- removed net N$4: C536.1, D523.C, R560.1
- removed net N$5: C537.1, R560.2, R561.2
- removed net N$6: C1.1, C538.2, L5.2, Q509.1
- removed net N$9: D523.A, Q524.1, R559.2
- new net N$26: VR63.A
- net +12V: now also GU.4; no longer C538.1, L5.1, R559.1, R681.2, TB.5, VR63.A
- net GND: now also GU.5; no longer C536.2, Q509.3, Q524.3, R555.2, R556.2, R562.1, TB.6
- net N$11: now also GU.2; no longer TB.2
- net N$17: no longer C537.2
- net N$20: no longer C534.1
- net N$24: now also GU.1; no longer TB.1
- net N$3: now also GU.3; no longer TB.4
- net N$46: no longer C535.1
- net N$7: now also GU.6; no longer TB.7
Routing:
- net GND: track 124.7 -> 82.6 mm
- net N$25: track 23.3 -> 0.00 mm
- net N$6: track 12.4 -> 0.00 mm
- net +12V: track 100.6 -> 91.0 mm
- net N$14: track 9.55 -> 0.00 mm
- net N$22: track 9.41 -> 0.00 mm
- net N$1: track 8.77 -> 0.00 mm
- net N$9: track 8.18 -> 0.00 mm
- net N$4: track 7.66 -> 0.00 mm
- net N$5: track 7.04 -> 0.00 mm
- net N$11: track 26.0 -> 19.1 mm
- net N$2: track 5.47 -> 0.00 mm
- net N$17: track 10.5 -> 5.18 mm
- net N$10: track 5.01 -> 0.00 mm
- net N$7: track 44.4 -> 39.8 mm
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